File: kicad/qrp-tester.kicad_pcb (KiCad board)
At the start: 2 copper layers, 80 x 23 mm, 33 parts, among them J1 IN, J2 PWR, Q1 MMBT3904, Q2 MMBT3904, Q3 MMBT3904, Q4 MMBT3904, SW1 ON/OFF, Y1 7023kHz

Commit message: Fix a connection bug.
Connections:
- C3 pad 2: Net-(C3-Pad1) -> Net-(C3-Pad2)
- C4 pad 1: Net-(C3-Pad1) -> Net-(C3-Pad2)
- Q1 pad 2: Net-(C3-Pad1) -> Net-(C3-Pad2)
- R3 pad 1: Net-(C3-Pad1) -> Net-(C3-Pad2)
Routing:
- net Net-(C3-Pad2): track 0.00 -> 14.1 mm
Other:
- board text added: "QRP Tester v01 - 20201024 - Design: K1MBO / Layout: BG1REN"
- board text removed: "QRP Tester v01 - 20201023 - Design: K1MBO / Layout: BG1REN"
